File: Eagle Files - PCB/Mutant.brd (EAGLE design)
At the start: 65.3 x 106.4 mm, 28 parts, among them M1 ARDUINO-NANO-3.0

Commit message: Code updated - Define buttons for rec and retrig swapped
Connections:
- net GND: now also C5.-
Changed lines of the file:
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@@
 <text x="18.034" y="49.3014" size="1.6764" layer="21" font="vector" ratio="28">MUTANT GENERATIVE SYNTH</text>
 <wire x1="17.399" y1="86.233" x2="49.911" y2="86.233" width="0.1524" layer="21"/>
-<dimension x1="19.0119" y1="69.977" x2="48.2981" y2="69.977" x3="33.655" y3="127" textsize="1.778" layer="20" dtype="horizontal"/>
-<dimension x1="17.399" y1="86.2203" x2="49.911" y2="81.9404" x3="33.655" y3="113.538" textsize="1.778" layer="20" dtype="horizontal"/>
 </plain>
 <attributes>
@@
 <contactref element="9V" pad="1"/>
 <contactref element="C3" pad="-"/>
+<contactref element="C5" pad="-"/>
 </signal>
 <signal name="+5V">
